File: arcboard-mk22-ffc.kicad_pcb (KiCad board)
At the start: 2 copper layers, 313 x 104.2 mm, 23 parts, among them J10 Conn_01x60, J7 Conn_01x04, J8 Conn_01x04

Commit message: fixing 0.3 footprint, the di-do mixup, and starting user comments updates
Connections:
- COL-0 pad 11: KEYS_DO -> Net-(COL-0-Pin_11)
- COL-0 pad 2: Net-(COL-0-Pin_2) -> KEYS_DO
- COL-1 pad 11: Net-(COL-0-Pin_2) -> Net-(COL-1-Pin_11)
- COL-1 pad 2: Net-(COL-1-Pin_2) -> Net-(COL-0-Pin_11)
- COL-2 pad 11: Net-(COL-1-Pin_2) -> Net-(COL-2-Pin_11)
- COL-2 pad 2: Net-(COL-2-Pin_2) -> Net-(COL-1-Pin_11)
- COL-5 pad 11: Net-(COL-4-Pin_2) -> KEYS_DI
- COL-5 pad 2: KEYS_DI -> Net-(COL-4-Pin_11)
- COL3 pad 11: Net-(COL-2-Pin_2) -> Net-(COL-4-Pin_2)
- COL3 pad 2: Net-(COL-4-Pin_11) -> Net-(COL-2-Pin_11)
Routing:
- net Net-(COL-2-Pin_2): track 126.1 -> 0.00 mm, vias 4 -> 0
- net Net-(COL-1-Pin_2): track 116.3 -> 0.00 mm, vias 6 -> 0
- net Net-(COL-2-Pin_11): track 0.00 -> 112.9 mm, vias 0 -> 4
- net Net-(COL-0-Pin_2): track 109.6 -> 0.00 mm, vias 2 -> 0
- net Net-(COL-1-Pin_11): track 0.00 -> 101.9 mm, vias 0 -> 4
- net Net-(COL-0-Pin_11): track 0.00 -> 97.3 mm, vias 0 -> 2
- net Net-(COL-4-Pin_11): track 127.9 -> 107.2 mm, vias 4 -> 1
- net ROW3: track 595.6 -> 609.0 mm
- net ROW4: track 645.9 -> 658.7 mm
- net KEYS_DI: track 291.3 -> 280.4 mm, vias 4 -> 2
- net Net-(COL-4-Pin_2): track 118.6 -> 129.0 mm, vias 0 -> 4
- net ROW0: track 1067.0 -> 1074.4 mm
- net KEYS_DO: track 505.1 -> 512.3 mm, vias 6 -> 8
- net +5V: track 2506.5 -> 2510.3 mm, vias 31 -> 33
- net ROW2: track 599.9 -> 603.0 mm
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